Commit message: finishing porting

File: franka_description/robots/common/franka_robot.xacro (robot description, xacro)
@@ -24,5 +24,5 @@
           <link name="${parent}" />
         </xacro:if>
-        <joint name="${parent}_joint" type="fixed">
+        <joint name="${parent}_franka_joint" type="fixed">
           <origin xyz="${xyz}" rpy="${rpy}" />
           <parent link="${parent}" />
